File: pcb/brushed-dual-esc.kicad_pcb (KiCad board)
At the start: 2 copper layers, 29.5 x 25 mm, 33 parts, among them J1 XT30PW-M, J2 TC2030-NL, J3 Conn_02x03_Odd_Even, J4 XT30PW-F, J5 XT30PW-F, U1 AZ1117-5.0, U2 TLV77133PDBVR, U3 STM32C011F4Ux, U4 DRV8231ADSGR, U5 DRV8231ADSGR

Commit message: Final commit
Routing:
- net /DRV1_ISENSE: vias 3 -> 2
