File: pcb/brushed-dual-esc.kicad_pcb (KiCad board)
At the start: 2 copper layers, 30 x 25 mm, 34 parts, among them J10 RX_CH2, J11 RX_CH1, J12 +5V, J13 GND, J2 TC2030-NL, J3 DRV1_OUT1, J5 DRV1_OUT2, J6 DRV2_OUT1, J7 DRV2_OUT2, J8 +BATT, J9 -BATT, U1 AZ1117CR-5.0TRG1, U2 TLV77133PDBVR, U3 STM32C011F6U6, U6 DRV8231ADDAR, U7 DRV8231ADDAR

Commit message: Make pretty
Parts:
- moved D2 0.75 mm to (156.2, 73.0)
- moved R6 0.75 mm to (158.2, 73.0)
Routing:
- net +3V3: track 48.1 -> 47.3 mm
- net GND: vias 45 -> 44
Other:
- board text added: "+"
- board text added: "-"
- board text added: "1"
- board text added: "2"
- board text added: "5V"
- board text added: "DRV1"
- board text added: "DRV2"
- board text added: "GND"
- board text added: "M2"
- board text added: "S1"
- board text added: "S2"
- board text added: "STATUS"
- board text added: "SWD"

Commit message: update front silkscreen
Other:
- board text added: "5V 1A"
- board text removed: "5V"
Changed lines of the file:
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@@
 		)
+	)
+	(gr_poly
+		(pts
+			(xy 149.25 64.5) (xy 149.25 63.8) (xy 148.6 63.8)
+		)
+		(stroke
+			(width 0.1)
+			(type solid)
+		)
+		(fill yes)
+		(layer "F.SilkS")
+	)
+	(gr_line
+		(start 145.75 64.5)
+		(end 145.75 70.25)
+		(stroke
+			(width 0.1)
+			(type default)
+		)
+		(layer "F.SilkS")
+	)
+	(gr_line
+		(start 145.75 70.25)
+		(end 149.25 70.25)
+		(stroke
+			(width 0.1)
+			(type default)
+		)
+		(layer "F.SilkS")
+	)
+	(gr_line
+		(start 146.5 63.75)
+		(end 145.75 64.5)
+		(stroke
+			(width 0.1)
+			(type default)
+		)
+		(layer "F.SilkS")
+	)
+	(gr_line
+		(start 148.5 63.75)
+		(end 146.5 63.75)
+		(stroke
+			(width 0.1)
+			(type default)
+		)
+		(layer "F.SilkS")
+	)
+	(gr_line
+		(start 148.5 63.75)
+		(end 150.6 63.75)
+		(stroke
+			(width 0.1)
+			(type default)
+		)
+		(layer "F.SilkS")
+	)
+	(gr_line
+		(start 149.25 64.5)
+		(end 148.5 63.75)
+		(stroke
+			(width 0.1)
+			(type default)
+		)
+		(layer "F.SilkS")
+	)
+	(gr_line
+		(start 149.25 70.25)
+		(end 149.25 64.5)
+		(stroke
+			(width 0.1)
+			(type default)
+		)
+		(layer "F.SilkS")
+	)
+	(gr_line
+		(start 150.6 63.75)
+		(end 150.6 66.8)
+		(stroke
+			(width 0.1)
+			(type default)
+		)
+		(layer "F.SilkS")
+	)
+	(gr_line
+		(start 150.6 66.8)
+		(end 149.3 66.8)
+		(stroke
+			(width 0.1)
+			(type default)
+		)
+		(layer "F.SilkS")
 	)
 	(gr_line
@@
 		)
 	)
-	(gr_text "5V"
+	(gr_text "5V 1A"
 		(at 151 72.5 90)
 		(layer "F.SilkS")
@@
 	)
 	(gr_text "SWD"
-		(at 149.5 67 90)
-		(layer "F.SilkS")
+		(at 149.4 65.25 90)
+		(layer "F.SilkS" knockout)
 		(effects
 			(font
@@
 	)
 	(gr_text "1"
-		(at 146.1 60.1 270)
+		(at 146.1 57 270)
 		(layer "F.SilkS")
 		(effects
@@
 	)
 	(gr_text "2"
-		(at 146.1 63.5 270)
-		(layer "F.SilkS")
-		(effects
+		(at 146.1 60.4 270)
+		(layer "F.SilkS")
+		(effects

Commit message: Add logo to back
Parts:
- added G***: LOGO, LOGO, B.Cu at (160.0, 62.5)
